File: bottom/bottom.kicad_sch (KiCad schematic)
At the start: 3 parts

Commit message: new rev
Parts:
- added H4: MountingHole, one:Hole_2.2mm, symbol Mechanical:MountingHole
- H1, H2, H3: value StandoffHole -> MountingHole
Changed lines of the file:
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@@
 (kicad_sch (version 20230121) (generator eeschema)
   (paper "A4")
-  (symbol (lib_id "Mechanical:MountingHole") (at 19.05 62.23 0) (unit 1)
+  (symbol (lib_id "Mechanical:MountingHole") (at 19.05 36.83 0) (unit 1)
     (in_bom yes) (on_board yes) (dnp no) (fields_autoplaced)
-    (property "Reference" "H3" (at 21.59 60.96 0)
+    (property "Reference" "H4" (at 21.59 35.56 0)
       (effects (font (size 1.27 1.27)) (justify left))
     )
-    (property "Value" "StandoffHole" (at 21.59 63.5 0)
+    (property "Value" "MountingHole" (at 21.59 38.1 0)
       (effects (font (size 1.27 1.27)) (justify left))
     )
-    (property "Footprint" "one:Hole_2.2mm" (at 19.05 62.23 0)
+    (property "Footprint" "one:Hole_2.2mm" (at 19.05 36.83 0)
       (effects (font (size 1.27 1.27)) hide)
     )
-    (property "Datasheet" "~" (at 19.05 62.23 0)
+    (property "Datasheet" "~" (at 19.05 36.83 0)
       (effects (font (size 1.27 1.27)) hide)
     )
     (instances
-      (project "shield"
+      (project "bottom"
+        (path "/1fd8269d-bfbb-4294-b901-abae7a95debd"
+          (reference "H4") (unit 1)
+        )
+      )
+    )
+  )
+  (symbol (lib_id "Mechanical:MountingHole") (at 19.05 26.67 0) (unit 1)
+    (in_bom yes) (on_board yes) (dnp no) (fields_autoplaced)
+    (property "Reference" "H2" (at 21.59 25.4 0)
+      (effects (font (size 1.27 1.27)) (justify left))
+    )
+    (property "Value" "MountingHole" (at 21.59 27.94 0)
+      (effects (font (size 1.27 1.27)) (justify left))
+    )
+    (property "Footprint" "one:Hole_2.2mm" (at 19.05 26.67 0)
+      (effects (font (size 1.27 1.27)) hide)
+    )
+    (property "Datasheet" "~" (at 19.05 26.67 0)
+      (effects (font (size 1.27 1.27)) hide)
+    )
+    (instances
+      (project "bottom"
+        (path "/1fd8269d-bfbb-4294-b901-abae7a95debd"
+          (reference "H2") (unit 1)
+        )
+      )
+    )
+  )
+  (symbol (lib_id "Mechanical:MountingHole") (at 19.05 31.75 0) (unit 1)
+    (in_bom yes) (on_board yes) (dnp no) (fields_autoplaced)
+    (property "Reference" "H3" (at 21.59 30.48 0)
+      (effects (font (size 1.27 1.27)) (justify left))
+    )
+    (property "Value" "MountingHole" (at 21.59 33.02 0)
+      (effects (font (size 1.27 1.27)) (justify left))
+    )
+    (property "Footprint" "one:Hole_2.2mm" (at 19.05 31.75 0)
+      (effects (font (size 1.27 1.27)) hide)
+    )
+    (property "Datasheet" "~" (at 19.05 31.75 0)
+      (effects (font (size 1.27 1.27)) hide)
+    )
+    (instances
+      (project "bottom"
         (path "/1fd8269d-bfbb-4294-b901-abae7a95debd"
           (reference "H3") (unit 1)
@@
     )
   )
-  (symbol (lib_id "Mechanical:MountingHole") (at 19.05 52.07 0) (unit 1)
+  (symbol (lib_id "Mechanical:MountingHole") (at 19.05 21.59 0) (unit 1)
     (in_bom yes) (on_board yes) (dnp no) (fields_autoplaced)
-    (property "Reference" "H1" (at 21.59 50.8 0)
+    (property "Reference" "H1" (at 21.59 20.32 0)
       (effects (font (size 1.27 1.27)) (justify left))
     )
-    (property "Value" "StandoffHole" (at 21.59 53.34 0)
+    (property "Value" "MountingHole" (at 21.59 22.86 0)
       (effects (font (size 1.27 1.27)) (justify left))
     )
-    (property "Footprint" "one:Hole_2.2mm" (at 19.05 52.07 0)
+    (property "Footprint" "one:Hole_2.2mm" (at 19.05 21.59 0)
       (effects (font (size 1.27 1.27)) hide)
     )
-    (property "Datasheet" "~" (at 19.05 52.07 0)
+    (property "Datasheet" "~" (at 19.05 21.59 0)
       (effects (font (size 1.27 1.27)) hide)
     )
     (instances
-      (project "shield"
+      (project "bottom"
         (path "/1fd8269d-bfbb-4294-b901-abae7a95debd"
           (reference "H1") (unit 1)
         )
       )
-    )
-  )
-  (symbol (lib_id "Mechanical:MountingHole") (at 19.05 57.15 0) (unit 1)
-    (in_bom yes) (on_board yes) (dnp no) (fields_autoplaced)
-    (property "Reference" "H2" (at 21.59 55.88 0)
-      (effects (font (size 1.27 1.27)) (justify left))
-    )
-    (property "Value" "StandoffHole" (at 21.59 58.42 0)
-      (effects (font (size 1.27 1.27)) (justify left))
-    )
-    (property "Footprint" "one:Hole_2.2mm" (at 19.05 57.15 0)
-      (effects (font (size 1.27 1.27)) hide)
-    )
-    (property "Datasheet" "~" (at 19.05 57.15 0)
-      (effects (font (size 1.27 1.27)) hide)
-    )
-    (instances
-      (project "shield"
-        (path "/1fd8269d-bfbb-4294-b901-abae7a95debd"
-          (reference "H2") (unit 1)
-        )
-      )
