File: pcb/pcb.kicad_sch (KiCad schematic)
At the start: 53 parts, among them J1 BATT, SW1 SW_SPST, SW10 SW_SPST, SW11 SW_SPST, SW12 SW_SPST, SW13 SW_SPST, SW14 SW_SPST, SW15 SW_SPST, SW16 SW_SPST, SW17 SW_SPST, SW18 SW_SPST, SW19 SW_SPST, SW2 SW_SPST, SW20 SW_SPST, SW21 SW_SPST, SW3 SW_SPST, SW4 SW_SPST, SW5 SW_SPST, SW6 SW_SPST, SW7 SW_SPST, SW8 SW_SPST, SW9 SW_SPST, U1 XIAO_nRF52840

Commit message: new rev
Parts:
- removed H5: MountingHole, s1:Hole_4.2mm, symbol Mechanical:MountingHole
- added J2: BATT, one:JST_SH_Battery_DUAL, symbol Connector:Conn_01x02_Pin
- D1, D10, D11, D12, D13, D14, D15, D16, D17, D18, D19, D2, D20, D21, D3, D4, D5, D6, D7, D8, D9: footprint s1:Diode_TH_SMD_DUAL -> one:Diode_TH_SMD_DUAL
- H1, H2, H3, H4: footprint s1:Hole_4.2mm -> one:Hole_4.2mm
- H6, H7, H8: footprint s1:Hole_2.2mm -> one:Hole_2.2mm
- J1: footprint s1:Battery -> one:Battery
- PWR1: footprint s1:MSK-12C02_DUAL -> one:MSK-12C02_DUAL
- SW1, SW10, SW11, SW12, SW13, SW14, SW15, SW16, SW17, SW18, SW19, SW2, SW20, SW21, SW3, SW4, SW5, SW6, SW7, SW8, SW9: footprint s1:KS-27_Cherry_MX_Hotswap_1U_DUAL -> one:KS-27_KS-33_Hotswap_1U_DUAL
- U1: footprint s1:XIAO_nRF52840_DUAL -> one:XIAO_nRF52840_DUAL; symbol s1:XIAO_nRF52840 -> one:XIAO_nRF52840
Connections:
- net B-: now also J2.2 (Pin_2)
- net at J1.1 (Pin_1), PWR1.2 (B): now also J2.1 (Pin_1)
