File: pcb/pcb.kicad_pcb (KiCad board)
At the start: 2 copper layers, 136 x 91.9 mm, 55 parts, among them J1 BATT, J2 BATT, SW1 SW_SPST, SW10 SW_SPST, SW11 SW_SPST, SW12 SW_SPST, SW13 SW_SPST, SW14 SW_SPST, SW15 SW_SPST, SW16 SW_SPST, SW17 SW_SPST, SW18 SW_SPST, SW19 SW_SPST, SW2 SW_SPST, SW20 SW_SPST, SW21 SW_SPST, SW3 SW_SPST, SW4 SW_SPST, SW5 SW_SPST, SW6 SW_SPST, SW7 SW_SPST, SW8 SW_SPST, SW9 SW_SPST, U1 XIAO_nRF52840

Commit message: preparation for release
Parts:
- PWR1: moved to B.Cu
- U1: moved to F.Cu
- moved J1 4.00 mm to (196.0, 78.1)
- turned PWR1 to 180 degrees
- turned U1 to 0 degrees
Routing:
- net R1: track 140.3 -> 161.3 mm, vias 10 -> 15
- net R2: track 155.1 -> 175.6 mm, vias 10 -> 16
- net R0: track 145.0 -> 165.5 mm, vias 12 -> 18
- net R3: track 127.3 -> 134.9 mm, vias 7 -> 10
- net Net-(D21-A): track 23.7 -> 28.2 mm, vias 2 -> 3
- net Net-(J1-Pin_1): track 44.5 -> 48.5 mm, vias 4 -> 5
- net Net-(D20-A): track 23.2 -> 27.2 mm, vias 2 -> 3
- net Net-(D9-A): track 21.8 -> 25.2 mm, vias 2 -> 3
- net Net-(D8-A): track 20.3 -> 23.7 mm, vias 2 -> 3
- net Net-(D7-A): track 21.8 -> 25.2 mm, vias 2 -> 3
- net Net-(D6-A): track 10.8 -> 14.2 mm, vias 2 -> 3
- net Net-(D5-A): track 11.4 -> 14.8 mm, vias 2 -> 3
- net Net-(D4-A): track 11.4 -> 14.8 mm, vias 2 -> 3
- net Net-(D3-A): track 11.4 -> 14.8 mm, vias 2 -> 3
- net Net-(D2-A): track 10.5 -> 14.0 mm, vias 2 -> 3
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
Commit message: release 1.1
Parts:
- added G***: LOGO, one:en_logo, F.Cu at (162.2, 115.0)
Other:
- board text added: "Ergonaut One v1.1 by yumagulovrn"
- board text removed: "Ergonaut One v1.0 by yumagulovrn"

Commit message: naming fixes
Parts:
- J2: moved to F.Cu
- turned J2 to -90 degrees
