File: pcb/pcb.kicad_pcb (KiCad board)
At the start: 2 copper layers, 136 x 91.7 mm, 56 parts, among them J1 BATT, J2 BATT, SW1 SW_SPST, SW10 SW_SPST, SW11 SW_SPST, SW12 SW_SPST, SW13 SW_SPST, SW14 SW_SPST, SW15 SW_SPST, SW16 SW_SPST, SW17 SW_SPST, SW18 SW_SPST, SW19 SW_SPST, SW2 SW_SPST, SW20 SW_SPST, SW21 SW_SPST, SW3 SW_SPST, SW4 SW_SPST, SW5 SW_SPST, SW6 SW_SPST, SW7 SW_SPST, SW8 SW_SPST, SW9 SW_SPST, U1 XIAO_nRF52840

Commit message: feat: bump board version
Other:
- board text added: "Ergonaut One v1.2 by yumagulovrn"
- board text removed: "Ergonaut One v1.1 by yumagulovrn"
Changed lines of the file:
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@@
   (gr_circle (center 103.5 104.99097) (end 104.5 104.99097)
     (stroke (width 0.2) (type solid)) (fill none) (layer "User.9"))
-  (gr_text "Ergonaut One v1.1\nby yumagulovrn" (at 122.5 111.74097) (layer "B.SilkS")
+  (gr_text "Ergonaut One v1.2\nby yumagulovrn" (at 122.5 111.74097) (layer "B.SilkS")
     (effects (font (size 1 1) (thickness 0.2) bold) (justify mirror))
   )
@@
     (effects (font (size 1 1) (thickness 0.2) bold) (justify mirror))
   )
-  (gr_text "Ergonaut One v1.1\nby yumagulovrn" (at 122.5 111.74097) (layer "F.SilkS")
+  (gr_text "Ergonaut One v1.2\nby yumagulovrn" (at 122.5 111.74097) (layer "F.SilkS")
     (effects (font (size 1 1) (thickness 0.2) bold))
   )
