File: plate/plate.kicad_pcb (KiCad board)
At the start: 2 copper layers, 129.6 x 93.1 mm, 26 parts, among them SW1 SW_SPST, SW10 SW_SPST, SW11 SW_SPST, SW12 SW_SPST, SW13 SW_SPST, SW14 SW_SPST, SW15 SW_SPST, SW16 SW_SPST, SW17 SW_SPST, SW18 SW_SPST, SW19 SW_SPST, SW2 SW_SPST, SW20 SW_SPST, SW21 SW_SPST, SW3 SW_SPST, SW4 SW_SPST, SW5 SW_SPST, SW6 SW_SPST, SW7 SW_SPST, SW8 SW_SPST, SW9 SW_SPST

Commit message: new rev
Parts:
- removed H5: MountingHole, s1:Hole_2.2mm
- H1, H2, H3, H4: footprint s1:Hole_2.2mm -> one:Hole_2.2mm
- SW1, SW10, SW11, SW12, SW13, SW14, SW15, SW16, SW17, SW18, SW19, SW2, SW20, SW21, SW3, SW4, SW5, SW6, SW7, SW8, SW9: footprint s1:KS-27_Cherry_MX_Plate_Cutout -> one:KS-27_Cherry_MX_Plate_Cutout
- moved SW15 87.1 mm to (160.5, 62.2)
- moved SW2 53.9 mm to (122.5, 100.2)
- moved H4 50.5 mm to (186.2, 116.5)
- moved SW1 50.4 mm to (84.5, 67.0)
- moved SW14 46.6 mm to (122.5, 62.2)
- moved SW5 44.9 mm to (179.5, 102.6)
- moved SW4 44.9 mm to (179.5, 83.6)
- moved SW7 44.9 mm to (84.5, 86.0)
- moved SW10 44.7 mm to (141.5, 78.9)
- moved SW3 40.2 mm to (179.5, 64.6)
- moved SW9 28.5 mm to (141.5, 59.9)
- moved SW16 25.4 mm to (160.5, 81.2)
- moved SW17 25.4 mm to (160.5, 100.2)
- moved SW11 24.0 mm to (151.0, 119.7)
- moved SW18 23.7 mm to (141.5, 97.9)
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Other:
- board size 129.6 x 93.1 mm -> 129.4 x 92.9 mm
