File: plate/plate.kicad_sch (KiCad schematic)
At the start: 29 parts, among them SW1 SW_SPST, SW10 SW_SPST, SW11 SW_SPST, SW12 SW_SPST, SW13 SW_SPST, SW14 SW_SPST, SW15 SW_SPST, SW16 SW_SPST, SW17 SW_SPST, SW18 SW_SPST, SW19 SW_SPST, SW2 SW_SPST, SW20 SW_SPST, SW21 SW_SPST, SW3 SW_SPST, SW4 SW_SPST, SW5 SW_SPST, SW6 SW_SPST, SW7 SW_SPST, SW8 SW_SPST, SW9 SW_SPST

Commit message: new rev
Parts:
- removed H5: MountingHole, s1:Hole_2.2mm, symbol Mechanical:MountingHole
- removed H6, H7, H8: AlignmentHole, s1:Hole_1.0mm, symbol Mechanical:MountingHole
- H1, H2, H3, H4: footprint s1:Hole_2.2mm -> one:Hole_2.2mm
- SW1, SW10, SW11, SW12, SW13, SW14, SW15, SW16, SW17, SW18, SW19, SW2, SW20, SW21, SW3, SW4, SW5, SW6, SW7, SW8, SW9: footprint s1:KS-27_Cherry_MX_Plate_Cutout -> one:KS-27_Cherry_MX_Plate_Cutout
